File: maker-faire-badge.kicad_pcb (KiCad board)
At the start: 2 copper layers, 101.6 x 18.8 mm, 38 parts, among them J1 USB-C, Q1 2N3906, Q2 2N3906, Q3 2N3906, Q4 2N3906, Q5 2N3906, Q6 2N3906

Commit message: updated design files
Parts:
- BT1, BT2: value Battery_Cell -> ${REFERENCE}
- R1: value 59.2k -> 15.4k
- R10: value 40.2k -> 14k
- R12: value 14k -> 40.2k
- R3: value 15.4k -> 59.2k
- R4: value 48.7k -> 14.7k
- R6: value 14.7k -> 48.7k
- moved D2 22.2 mm to (159.0, 73.7)
- moved D4 22.2 mm to (150.4, 83.9)
- moved R16 22.2 mm to (135.9, 84.5)
- moved R17 22.2 mm to (159.0, 83.8)
- moved R9 22.2 mm to (135.9, 79.4)
- moved C1 22.2 mm to (99.1, 72.9)
- moved C2 22.2 mm to (99.1, 78.7)
- moved H1 22.2 mm to (104.1, 83.4)
- moved Q1 22.2 mm to (88.6, 72.9)
- moved Q2 22.2 mm to (88.6, 78.7)
- moved Q3 22.2 mm to (108.0, 72.9)
- moved Q4 22.2 mm to (108.0, 78.7)
- moved REF** 22.2 mm to (93.7, 84.1)
- moved C3 22.2 mm to (118.4, 72.9)
- moved C4 22.2 mm to (118.4, 78.7)
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Connections:
- net blue-led renamed LED-3
- net green-led renamed LED-2
- net red-led renamed LED-1
- C1 pad 1: base-2 -> BASE-1B
- C2 pad 1: base-1 -> BASE-1A
- C3 pad 1: base-4 -> BASE-2B
- C4 pad 1: base-3 -> BASE-2A
- C5 pad 1: base-6 -> BASE-3B
- C6 pad 1: base-5 -> BASE-3A
- Q1 pad 2: base-1 -> BASE-1A
- Q2 pad 2: base-2 -> BASE-1B
- Q3 pad 2: base-3 -> BASE-2A
- Q4 pad 2: base-4 -> BASE-2B
- Q5 pad 2: base-5 -> BASE-3A
- Q6 pad 2: base-6 -> BASE-3B
- R1 pad 1: base-2 -> GND
- R1 pad 2: GND -> BASE-1B
- R10 pad 1: base-6 -> GND
- R10 pad 2: GND -> BASE-3B
- R11 pad 1: Net-(Q5-C) -> GND
- R11 pad 2: GND -> Net-(Q5-C)
- R12 pad 1: base-5 -> GND
- R12 pad 2: GND -> BASE-3A
- R2 pad 1: Net-(Q1-C) -> GND
- R2 pad 2: GND -> Net-(Q1-C)
- R3 pad 1: base-1 -> GND
- R3 pad 2: GND -> BASE-1A
- R4 pad 1: base-4 -> GND
- R4 pad 2: GND -> BASE-2B
- R5 pad 1: Net-(Q3-C) -> GND
- R5 pad 2: GND -> Net-(Q3-C)
- R6 pad 1: base-3 -> GND
- R6 pad 2: GND -> BASE-2A
Routing:
- net base-6: track 22.9 -> 0.00 mm
- net BASE-1B: track 0.00 -> 22.9 mm
- net BASE-2B: track 0.00 -> 22.9 mm
- net base-4: track 22.9 -> 0.00 mm
- net base-2: track 22.9 -> 0.00 mm
- net BASE-3B: track 0.00 -> 22.9 mm
- net BASE-2A: track 0.00 -> 16.5 mm
- net base-5: track 16.5 -> 0.00 mm
- net base-3: track 16.5 -> 0.00 mm
- net BASE-1A: track 0.00 -> 16.5 mm
- net base-1: track 16.5 -> 0.00 mm
- net BASE-3A: track 0.00 -> 16.5 mm
Other:
- board text added: "1. Customer is to be contacted if one or more items listed below are in violation. 2. Design is a 2 layer board with a copper weight of 1 oz. 3. Board thickness is 1.6 mm 4. All trace widths are 6 mils or greater in the current design. 5. All trace clearances are 6 mils or greater in the current design. 6. PCB revision is on the bottom layer of copper as noted. Revision text is mirrored on this d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"
- board text added: "1. When possible, reference designators were placed within components. 2. 3 tables are included on the assembly drawing as follows: A. The component population that will set a color of D1 to either blink or stay solidly lit. B. The component population that will change the blink rate of a color of D1 when that color is set to blink. C. The component population that will set the power input config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"
- board text added: "ASSEMBLY NOTES"
- board text added: "BLINK LED 1"
- board text added: "BLINK LED 2"
- board text added: "BLINK LED 3"
- board text added: "DESIGNED BY 237 DECIMAL TO HEX"
- board text added: "LED SOLID BLINK 1 R15 R8 2 R14 R7 3 R16 R9"
- board text added: "LEDS 1,2,3 SOLID/BLINK"
- board text added: "REMOVE BATTERY BEFORE CONNECTING THE USB"
- board text added: "REV B"
- board text added: "Space for Manufacturer Markings on bottom side of board"
- board text added: "THE BATTERY OVERRIDES USB POWER"
- board text removed: "10.00 mils"
- board text removed: "2"
- board text removed: "4000.00 mils x 1090.00 mils"
- board text removed: "62.99 mils"
- board text removed: "7.00 mils / 7.00 mils"
- board text removed: "BLINK BLUE"
- board text removed: "BLINK GREEN"
- board text removed: "BLINK RED"
- board text removed: "BOARD CHARACTERISTICS"
- board text removed: "Board Thickness:"
- board text removed: "Board overall dimensions:"
- board text removed: "Castellated pads:"
- board text removed: "Copper Finish:"
- board text removed: "Copper Layer Count:"
- board text removed: "Edge card connectors:"
- board text removed: "HAL lead-free"
- board text removed: "Impedance Control:"
- board text removed: "Min hole diameter:"
- board text removed: "Min track/spacing:"
- board text removed: "NO BLINK LED R14 GREEN R15 RED R16 BLUE"
- board text removed: "No"
- board text removed: "Plated Board Edge:"
- board text removed: "REMOVE BATTERY BEFORE USING THE USB, THE BATTERY WILL DISCONNECT USB"
- board text removed: "REV A"
