File: maker-faire-badge.kicad_sch (KiCad schematic)
At the start: 45 parts, among them J1 USB-C, Q1 2N3906, Q2 2N3906, Q3 2N3906, Q4 2N3906, Q5 2N3906, Q6 2N3906

Commit message: BOM and Fabrication Note corrections
Parts:
- R1, R13, R15, R3: value 205 -> 82; PartNumber MFR-25FBF52-205R -> CFR-25JB-52-82R
- R10, R12, R8: value 95.3 -> 150; PartNumber MFR-25FBF52-95R3 -> CFR-25JB-52-150R
- R11, R7, R9: value 205 -> 150; PartNumber MFR-25FBF52-205R -> CFR-25JB-52-150R
- R14, R16, R2, R4: value 95.3 -> 82; PartNumber MFR-25FBF52-95R3 -> CFR-25JB-52-82R
- R17, R5: value 133 -> 82; PartNumber MFR-25FBF52-133R -> CFR-25JB-52-82R
- R18, R6: value 24.9 -> 82; PartNumber MFR-25FBF52-24R9 -> CFR-25JB-52-82R
- R19, R20: PartNumber MFR-25FBF52-5K1 -> CFR-25JB-52-5K1
- R21, R24, R27: value 261 -> 270; PartNumber MFR-25FBF52-261R -> CFR-25JB-52-270R
- R22: Manufacturer YAGEO -> Yageo; PartNumber CFR-25JR-52-82K -> CFR-25JB-52-82k
- R23: PartNumber CFR-25JR-52-30K -> CFR-25JB-52-30K
- R25: Manufacturer TE Connectivity -> Yageo; PartNumber CFR-25JR-52-150K -> CFR-25JB-52-150K
- R26, R29: Manufacturer Yageo -> Yageo; PartNumber CFR-25JR-52-30K -> CFR-25JB-52-30K
- R28: PartNumber CFR-25JR-52-110K -> CFR-25JB-52-110K
Other:
- title: Maker Faire Orange County Badge -> Maker Faire Orange County Acrylic Display
Changed lines of the file:
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@@
 	(paper "USLetter")
 	(title_block
-		(title "Maker Faire Orange County Badge")
+		(title "Maker Faire Orange County Acrylic Display")
 		(date "2025-10-26")
 		(rev "D")
@@
 			)
 		)
-		(property "Value" "95.3"
+		(property "Value" "82"
 			(at 204.47 156.21 90)
 			(effects
@@
 			)
 		)
-		(property "PartNumber" "MFR-25FBF52-95R3"
+		(property "PartNumber" "CFR-25JB-52-82R"
 			(at 204.47 160.02 0)
 			(effects
@@
 			)
 		)
-		(property "PartNumber" "MFR-25FBF52-5K1"
+		(property "PartNumber" "CFR-25JB-52-5K1"
 			(at 58.42 110.49 0)
 			(effects
@@
 			)
 		)
-		(property "Value" "95.3"
+		(property "Value" "82"
 			(at 204.47 143.51 90)
 			(effects
@@
 			)
 		)
-		(property "PartNumber" "MFR-25FBF52-95R3"
+		(property "PartNumber" "CFR-25JB-52-82R"
 			(at 204.47 147.32 0)
 			(effects
@@
 			)
 		)
-		(property "Value" "205"
+		(property "Value" "82"
 			(at 152.4 134.6199 0)
 			(effects
@@
 			)
 		)
-		(property "PartNumber" "MFR-25FBF52-205R"
+		(property "PartNumber" "CFR-25JB-52-82R"
 			(at 149.86 133.35 0)
 			(effects
@@
 			)
 		)
-		(property "Value" "205"
+		(property "Value" "82"
 			(at 246.38 134.6199 0)
 			(effects
@@
 			)
 		)
-		(property "PartNumber" "MFR-25FBF52-205R"
+		(property "PartNumber" "CFR-25JB-52-82R"
 			(at 243.84 133.35 0)
 			(effects
@@
 			)
 		)
-		(property "PartNumber" "CFR-25JR-52-30K"
+		(property "PartNumber" "CFR-25JB-52-30K"
 			(at 240.03 99.06 0)
 			(effects
@@
 			)
 		)
-		(property "Manufacturer" "Yageo"
+		(property "Manufacturer" "Yageo "
 			(at 240.03 99.06 0)
 			(effects
@@
 			)
 		)
-		(property "Value" "261"
+		(property "Value" "270"
 			(at 256.54 100.3299 0)
 			(effects
@@
 			)
 		)
-		(property "PartNumber" "MFR-25FBF52-261R"
+		(property "PartNumber" "CFR-25JB-52-270R"
 			(at 254 99.06 0)
 			(effects
@@
 			)
 		)
-		(property "PartNumber" "MFR-25FBF52-5K1"
+		(property "PartNumber" "CFR-25JB-52-5K1"
 			(at 71.12 110.49 0)
 			(effects
@@
 			)
 		)
-		(property "Value" "205"
+		(property "Value" "150"
 			(at 228.6 134.6199 0)
 			(effects
@@
 			)
 		)
-		(property "PartNumber" "MFR-25FBF52-205R"
+		(property "PartNumber" "CFR-25JB-52-150R"
 			(at 226.06 133.35 0)
 			(effects
@@
 			)
 		)
-		(property "Manufacturer" "TE Connectivity"
+		(property "Manufacturer" "Yageo "
 			(at 110.49 60.96 0)
 			(effects
@@
 			)
 		)
-		(property "PartNumber" "CFR-25JR-52-150K"
+		(property "PartNumber" "CFR-25JB-52-150K"
 			(at 110.49 60.96 0)
 			(effects
@@
 			)
 		)
-		(property "Value" "261"
+		(property "Value" "270"
 			(at 139.7 100.3299 0)
 			(effects
@@
 			)
 		)
-		(property "PartNumber" "MFR-25FBF52-261R"
+		(property "PartNumber" "CFR-25JB-52-270R"
 			(at 137.16 99.06 0)
 			(effects
@@
 			)
 		)
-		(property "Value" "205"
+		(property "Value" "82"
 			(at 161.29 134.6199 0)
 			(effects
@@
 			)
 		)
-		(property "PartNumber" "MFR-25FBF52-205R"
+		(property "PartNumber" "CFR-25JB-52-82R"
 			(at 158.75 133.35 0)
 			(effects
@@
 			)
 		)
-		(property "Value" "133"
+		(property "Value" "82"
 			(at 77.47 158.7499 0)
 			(effects
@@
 			)
 		)
-		(property "PartNumber" "MFR-25FBF52-133R"
+		(property "PartNumber" "CFR-25JB-52-82R"
 			(at 74.93 157.48 0)
 			(effects
@@
 			)
 		)
-		(property "Value" "95.3"
+		(property "Value" "150"
 			(at 119.38 130.81 90)
 			(effects
@@
 			)
 		)
-		(property "PartNumber" "MFR-25FBF52-95R3"
+		(property "PartNumber" "CFR-25JB-52-150R"
 			(at 119.38 134.62 0)
 			(effects
@@
 			)
 		)
-		(property "Value" "95.3"
+		(property "Value" "82"
 			(at 119.38 143.51 90)
 			(effects
@@
 			)
 		)
-		(property "PartNumber" "MFR-25FBF52-95R3"
+		(property "PartNumber" "CFR-25JB-52-82R"
 			(at 119.38 147.32 0)
 			(effects
@@
 			)
 		)
-		(property "PartNumber" "CFR-25JR-52-110K"
+		(property "PartNumber" "CFR-25JB-52-110K"
 			(at 227.33 60.96 0)
 			(effects
@@
 			)
 		)
-		(property "Value" "133"
+		(property "Value" "82"
 			(at 68.58 158.7499 0)
 			(effects
@@
 			)
 		)
-		(property "PartNumber" "MFR-25FBF52-133R"
+		(property "PartNumber" "CFR-25JB-52-82R"
 			(at 66.04 157.48 0)
 			(effects
@@
 			)
 		)
-		(property "Value" "205"
+		(property "Value" "150"
 			(at 59.69 158.7499 0)
 			(effects
@@
 			)
 		)
-		(property "PartNumber" "MFR-25FBF52-205R"
+		(property "PartNumber" "CFR-25JB-52-150R"
 			(at 57.15 157.48 0)
 			(effects
@@
 			)
 		)
-		(property "Value" "24.9"
+		(property "Value" "82"
 			(at 35.56 167.64 90)
 			(effects
@@
 			)
 		)
-		(property "PartNumber" "MFR-25FBF52-24R9"
+		(property "PartNumber" "CFR-25JB-52-82R"
 			(at 35.56 171.45 0)
 			(effects
@@
 			)
 		)
-		(property "Value" "205"
+		(property "Value" "150"
 			(at 143.51 134.6199 0)
 			(effects
@@
 			)
 		)
-		(property "PartNumber" "MFR-25FBF52-205R"
+		(property "PartNumber" "CFR-25JB-52-150R"
 			(at 140.97 133.35 0)
 			(effects
@@
 			)
 		)
-		(property "Value" "95.3"
+		(property "Value" "82"
 			(at 119.38 156.21 90)
 			(effects
@@
 			)
 		)
-		(property "PartNumber" "MFR-25FBF52-95R3"
+		(property "PartNumber" "CFR-25JB-52-82R"
 			(at 119.38 160.02 0)
 			(effects
@@
 			)
 		)
-		(property "Value" "95.3"
+		(property "Value" "150"
 			(at 204.47 130.81 90)
 			(effects
@@
 			)
 		)
-		(property "PartNumber" "MFR-25FBF52-95R3"
+		(property "PartNumber" "CFR-25JB-52-150R"
 			(at 204.47 134.62 0)
 			(effects
@@
 			)
 		)
-		(property "PartNumber" "CFR-25JR-52-30K"
+		(property "PartNumber" "CFR-25JB-52-30K"
 			(at 181.61 99.06 0)
 			(effects
@@
 			)
 		)
-		(property "Manufacturer" "YAGEO"
+		(property "Manufacturer" "Yageo"
 			(at 168.91 60.96 0)
 			(effects
@@
 			)
 		)
-		(property "PartNumber" "CFR-25JR-52-82K"
+		(property "PartNumber" "CFR-25JB-52-82k"
 			(at 168.91 60.96 0)
 			(effects
@@
 			)
 		)
-		(property "Value" "95.3"
+		(property "Value" "150"
 			(at 35.56 154.94 90)
 			(effects
@@
 			)
 		)
-		(property "PartNumber" "MFR-25FBF52-95R3"
+		(property "PartNumber" "CFR-25JB-52-150R"
 			(at 35.56 158.75 0)
 			(effects
@@
 			)
 		)
-		(property "Value" "205"
+		(property "Value" "82"
 			(at 237.49 134.6199 0)
 			(effects
@@
 			)
 		)
-		(property "PartNumber" "MFR-25FBF52-205R"
+		(property "PartNumber" "CFR-25JB-52-82R"
 			(at 234.95 133.35 0)
 			(effects
@@
 			)
 		)
-		(property "Value" "24.9"
+		(property "Value" "82"
 			(at 35.56 180.34 90)
 			(effects
@@
 			)
 		)
-		(property "PartNumber" "MFR-25FBF52-24R9"
+		(property "PartNumber" "CFR-25JB-52-82R"
 			(at 35.56 184.15 0)
 			(effects
@@
 			)
 		)
-		(property "Manufacturer" "Yageo"
+		(property "Manufacturer" "Yageo "
 			(at 123.19 99.06 0)
 			(effects
@@
 			)
 		)
-		(property "PartNumber" "CFR-25JR-52-30K"
+		(property "PartNumber" "CFR-25JB-52-30K"
 			(at 123.19 99.06 0)
 			(effects
@@
 			)
 		)
-		(property "Value" "261"
+		(property "Value" "270"
 			(at 198.12 100.3299 0)
 			(effects
@@
 			)
 		)
-		(property "PartNumber" "MFR-25FBF52-261R"
+		(property "PartNumber" "CFR-25JB-52-270R"
 			(at 195.58 99.06 0)
 			(effects
